File: shieldRF/shieldRF.sch (KiCad schematic (older format))
At the start: 0 parts

Commit message: Update en esquemático
Se avanzó sobre el esquemático, lo que incluyó incorporación de nuevas librerías.
Parts:
- added ANT: Antenna, symbol Antenna
- added C1: 22uF, symbol C
- added C2, C3, C4, C5, C6: 104pF, symbol C
- added D2: LED_ALT, symbol LED_ALT
- added IC2: AP111733, TO_SOT_Packages_SMD:SOT-223, symbol AP111733
- added IC3: SN74LVC1G125DCKR, SC-70-5, symbol LOGIC-SN74LVC1G125DCKR(SC70-5)
- added IC4: H5V3G, symbol H5V3G
- added R2, R3: 1K, symbol R
- added R4: 22, symbol R
- added S1: SW_SPDT, symbol SW_SPDT
- added U?: XBee_Header, symbol XBee_Header
Connections:
- new net: IC3.2 (A), R3.1
- new net: IC3.4 (Y), U?.3 (DIN/~CONFIG)
- new net: ANT.1 (A), IC4.1 (ANT)
- new net: R2.1, U?.15 (Assoc./AD5/DIO5)
- new net: R4.2, U?.2 (DOUT)
- new net: R4.1, S1.1 (A)
- new net: D2.2 (A), R2.2
- new net +3.3V: C3.1, C4.1, C5.1, IC2.2 (VO), IC2.4 (VO), IC3.5 (VCC), U?.1 (VCC)
- new net +5V: C1.1, C2.1, C6.1, IC2.3 (VI), IC4.3 (VCC)
- new net GND: C1.2, C2.2, C3.2, C4.2, C5.2, C6.2, D2.1 (K), IC2.1 (GND/ADJ), IC3.1 (!OE!), IC3.3 (GND), IC4.2 (GND), IC4.6 (GND), U?.10 (GND)
